File: Engine_cables_VAG.kicad_sch (KiCad schematic)
At the start: 2 parts, among them J2 ECU_Con, J2 Lambda1

Commit message: Is this an OK foundation for further work?
Parts:
- removed J2: ECU_Con, symbol Connectors:ECU_Connector_ME7.5
- added J1: T121, symbol bosch_me7_5_t121:T121
- added J3: Conn_01x05, symbol Connector_Generic:Conn_01x05
- added J5, J6, J7, J8: Conn_01x4-pin, symbol Connector_Generic:Conn_01x04
- added K1, K2: DIPxx-1Axx-12xD, Relay_THT:Relay_StandexMeder_DIP_LowProfile, symbol Relay:DIPxx-1Axx-12xD
- J2: value Lambda1 -> Conn_01x05; symbol Connector:Conn_01x05_Pin -> Connector_Generic:Conn_01x05
Connections:
- net Heater+ renamed LSU1.Heater+
- net Heater- renamed LSU1.Heater-
- net Nernst_cell_voltage renamed LSU1.Nernst_cell_voltage
- net Pump_current renamed LSU1.Pump_current
- net Virtual_ground renamed LSU1.Virtual_ground
- new net: K1.1, K1.14
- new net: K1.13, K1.2
- new net: J1.21 (Relay_Contr), K1.6
- new net: K1.7, K1.8
- new net: J1.65 (Fuel_pump_relay), K2.6
- new net: K2.1, K2.14
- new net: K2.13, K2.2
- new net: K2.7, K2.8
- new net +BATT: J1.62 (Bat_perm)
- new net Coil1.12V: J5.1 (Pin_1)
- new net Coil1.GND: J5.2 (Pin_2)
- new net Coil1.Signal: J1.102 (IgnCoil_1), J5.3 (Pin_3)
- new net Coil2.12V: J6.1 (Pin_1)
- new net Coil2.GND: J6.2 (Pin_2)
- new net Coil2.Signal: J1.95 (IgnCoil_3), J6.3 (Pin_3)
- new net Coil3.Signal: J1.103 (IgnCoil_3)
- new net Coil4.Signal: J1.94 (IgnCoil_4)
- new net GND: J5.4 (Pin_4), J6.4 (Pin_4), J7.4 (Pin_4), J8.4 (Pin_4)
Other:
- added sheet Ignition Doc (Ignition.kicad_sch)
- note added: "Alternator"
- note added: "Crank angle"
- note added: "DBW throttel body"
- note added: "Ignition Coils"
- note added: "Ignition cable bundle"
- note added: "Injectors"
- note added: "LSUs (O2 sensors)"
- note added: "MAF"
- note added: "Starter"
- note added: "VVT"
